File: stereoBoy/stereoBoy_MGB.kicad_pcb (KiCad board)
At the start: 4 copper layers, 69.6 x 114.8 mm, 119 parts, among them J1 Conn_01x02, J3 GameBoy_Cartridge, J4 Conn_01x04, J5 SJ1-3524N, J7 USB_C_Receptacle_USB2.0_16P, J9 Conn_01x06, Q1 DMG2301L, Q2 MMUN2133LT1, SW1 MGB-SW1, U1 CODECODER-VS1053B_LQFP48_, U10 MCP73871, U11 TPS61091, U15 AP2112K-3.3, U16 PAM8302AAD, U2 RP2040, U5 TS5A23159DGS, U6 TEA5767, U7 TS5A23159DGS, Y1 12M, Y2 12M

Commit message: redesigned PSU for AAAs
Parts:
- removed C17: 10uF, SparkFun-Capacitor:C_0805_2012Metric
- removed C18, C29: 4.7uF, SparkFun-Capacitor:C_0805_2012Metric
- removed C19, C20, C24, C27: 0.1uF, SparkFun-Capacitor:C_0805_2012Metric
- removed C21: 100uF, SparkFun-Capacitor:C_0805_2012Metric
- removed C22: 10uF, Capacitor_SMD:C_0603_1608Metric
- removed C23, C26: 4.7uF, SparkFun-Capacitor:C_0603_1608Metric
- removed C25: 0.1uF, Capacitor_SMD:C_0805_2012Metric
- removed C28: 10uF, SparkFun-Capacitor:C_0603_1608Metric
- removed C32: 4.7uF, Capacitor_SMD:C_0805_2012Metric
- removed D20, D21: Green, SparkFun-LED:LED_0603_1608Metric_Green
- removed J1: Conn_01x02, Connector_JST:JST_PH_S2B-PH-K_1x02_P2.00mm_Horizontal
- removed R17, R18, R19, R20, R21, R22, R23, R24, R25, R26, R27, R28, R29: 1k, SparkFun-Resistor:R_0603_1608Metric
- removed U10: MCP73871, Package_DFN_QFN:QFN-20-1EP_4x4mm_P0.5mm_EP2.5x2.5mm
- removed U11: TPS61091, Package_DFN_QFN:Texas_RSA_VQFN-16-1EP_4x4mm_P0.65mm_EP2.7x2.7mm_ThermalVias
- removed U15: AP2112K-3.3, Package_TO_SOT_SMD:SOT-23-5
- added +0: MGB+BATTERY4, MGBC-MBL-01_2_1:MGB+BATTERY4, F.Cu at (137.8, 117.9)
- added -0: MGB-BATTERY4, MGBC-MBL-01_2_1:MGB-BATTERY4, F.Cu at (129.7, 137.1)
- added C10: 1.0uF, SparkFun-Capacitor:C_0805_2012Metric, F.Cu at (124.5, 127.2)
- added C7: 1.0uF, SparkFun-Capacitor:C_0805_2012Metric, F.Cu at (117.8, 128.0)
- added C8: 1.0uF, SparkFun-Capacitor:C_0805_2012Metric, F.Cu at (121.5, 132.2)
- added C9: 1.0uF, SparkFun-Capacitor:C_0805_2012Metric, F.Cu at (121.5, 130.2)
- added R1: 1.07M, SparkFun-Resistor:R_0603_1608Metric, F.Cu at (124.8, 121.5)
- added R13: 340k, SparkFun-Resistor:R_0603_1608Metric, F.Cu at (117.8, 126.2)
- added R16: 330, SparkFun-Resistor:R_0603_1608Metric, F.Cu at (115.2, 124.0)
- added R3: 340k, SparkFun-Resistor:R_0603_1608Metric, F.Cu at (124.2, 123.8)
- added R4: 1.07M, SparkFun-Resistor:R_0603_1608Metric, F.Cu at (117.0, 124.0)
- added U3: TPS61090, Package_DFN_QFN:Texas_RSA_VQFN-16-1EP_4x4mm_P0.65mm_EP2.7x2.7mm_ThermalVias, F.Cu at (120.5, 123.2)
- added U4: AP2112K-3.3, Package_TO_SOT_SMD:SOT-23-5, F.Cu at (121.5, 127.5)
- D19: value Green -> LED; footprint SparkFun-LED:LED_0603_1608Metric_Green -> SparkFun-LED:LED_0603_1608Metric
- Q2: value MMUN2133LT1 -> MMUN2133LT1G; footprint Package_TO_SOT_SMD:SOT-23 -> MMUN2133LT1G:SOT95P240X111-3N
- moved ZOOM_CAP1 247.8 mm to (101.8, 131.2)
- moved Q2 17.9 mm to (116.0, 120.2), turned to 90 degrees
- moved L1 2.87 mm to (122.2, 116.8), turned to 180 degrees
- moved D19 1.50 mm to (115.2, 127.0), turned to 90 degrees
- moved C1 0.39 mm to (144.6, 96.3)
- moved C2 0.39 mm to (139.5, 96.3)
- moved C3 0.39 mm to (155.0, 98.2)
- moved C4 0.39 mm to (150.0, 98.2)
- moved C5 0.39 mm to (168.7, 89.9)
- moved C6 0.39 mm to (162.6, 89.9)
- moved U1 0.39 mm to (152.5, 91.5)
- moved U2 0.39 mm to (141.9, 90.4)
- moved Y1 0.39 mm to (142.0, 96.3)
- moved Y2 0.39 mm to (152.5, 98.2)
Connections:
- net VBAT renamed +BATT
- D19 pad 1: Net-(D19-K) -> GND
Routing:
- net +5V: track 43.5 -> 0.00 mm
- net +BATT: track 35.9 -> 0.00 mm
- net VLIPO: track 16.6 -> 0.00 mm
- net Net-(L1-Pad2): track 8.07 -> 0.00 mm
- net Net-(Q2-B): track 6.12 -> 0.00 mm
- net Net-(U11-LBI): track 4.68 -> 0.00 mm
- net Net-(U10-VPCC): track 3.18 -> 0.00 mm
- net Net-(D20-K): track 2.89 -> 0.00 mm
- net Net-(U10-THERM): track 2.86 -> 0.00 mm
- net Net-(U11-FB): track 2.70 -> 0.00 mm
- net Net-(D19-K): track 2.43 -> 0.00 mm
- net Net-(U10-PROG3): track 2.35 -> 0.00 mm
- net Net-(Q2-C): track 1.83 -> 0.00 mm
- net Net-(U11-EN): track 1.77 -> 0.00 mm
- net Net-(U10-PROG1): track 1.66 -> 0.00 mm
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
Commit message: yeah
Parts:
- removed BTN_SR1: 74HC165, Package_SO:SOIC-16_3.9x9.9mm_P1.27mm
- removed J4: Conn_01x04, Connector_PinHeader_2.54mm:PinHeader_1x04_P2.54mm_Vertical
- removed J9: Conn_01x06, SparkFun-Connector:1x06
- removed SW_BOOT1, SW_NRST1: SMD_4.2x3.2mm_h2.5mm, SparkFun-Switch:Push_SMD_4.2x3.2mm
- removed Y1: 12M, SparkFun-Clock:Crystal_SMD_3.2x1.5mm
- added 1.54_IPS_LCD: 1.54_IPS_LCD, 1.54_IPS_LCD_Adafruit:1.54_IPS_LCD, B.Cu at (155.9, 70.6)
- added C11: 1.0uF, SparkFun-Capacitor:C_0805_2012Metric, B.Cu at (171.4, 152.2)
- added C12: 1.0uF, SparkFun-Capacitor:C_0805_2012Metric, B.Cu at (178.1, 158.3)
- added C13: 1.0uF, SparkFun-Capacitor:C_0805_2012Metric, F.Cu at (163.0, 78.5)
- added C14: 2.2uF, Capacitor_SMD:C_0402_1005Metric, F.Cu at (153.4, 78.8)
- added C15: 1.0uF, SparkFun-Capacitor:C_0805_2012Metric, B.Cu at (126.0, 94.3)
- added C17: 0.1uF, SparkFun-Capacitor:C_0402_1005Metric, F.Cu at (142.9, 83.4)
- added C18: 0.1uF, SparkFun-Capacitor:C_0402_1005Metric, F.Cu at (142.9, 87.4)
- added C19: 0.1uF, SparkFun-Capacitor:C_0402_1005Metric, F.Cu at (147.0, 92.1)
- added C20: 18pF, SparkFun-Capacitor:C_0402_1005Metric, F.Cu at (147.0, 94.0)
- added C21: 18pF, SparkFun-Capacitor:C_0402_1005Metric, F.Cu at (151.8, 94.0)
- added C22: 0.1uF, SparkFun-Capacitor:C_0402_1005Metric, F.Cu at (150.7, 92.1)
- added C23: 0.1uF, SparkFun-Capacitor:C_0402_1005Metric, F.Cu at (155.9, 85.3)
- added C24: 0.1uF, SparkFun-Capacitor:C_0402_1005Metric, F.Cu at (151.3, 78.6)
- added C25: 0.1uF, SparkFun-Capacitor:C_0402_1005Metric, F.Cu at (142.9, 85.3)
- added C26: 0.1uF, Capacitor_SMD:C_Elec_5x5.4, B.Cu at (149.4, 94.3)
- added C27: 0.1uF, Capacitor_SMD:C_Elec_5x5.4, B.Cu at (142.6, 94.3)
- added FB1: FerriteBead_Small, Inductor_SMD:L_0402_1005Metric, F.Cu at (152.4, 78.8)
- added J1: Conn_01x22_FPC_0.5mm, SparkFun-Connector:FPC_1x22_P0.5mm_Horizontal_BottomContact, F.Cu at (155.7, 66.1)
- added J2: JST_1mm_3_Vertical, SparkFun-Connector:JST_1x03_P1.0mm_Horizontal_SMD, B.Cu at (120.6, 92.2)
- added L2: 600 Ohm, SparkFun-Capacitor:C_0805_2012Metric, F.Cu at (160.3, 78.5)
- added L3: 600 Ohm, SparkFun-Capacitor:C_0805_2012Metric, F.Cu at (165.7, 78.5)
- added R17: 330, SparkFun-Resistor:R_0603_1608Metric, B.Cu at (175.9, 63.8)
- added R18: 330, SparkFun-Resistor:R_0603_1608Metric, B.Cu at (175.9, 62.2)
- added R19: 330, SparkFun-Resistor:R_0603_1608Metric, B.Cu at (175.9, 60.6)
- added R20: 1k, Resistor_SMD:R_0805_2012Metric, B.Cu at (174.0, 97.8)
- added R21: 1k, Resistor_SMD:R_0805_2012Metric, B.Cu at (174.0, 95.7)
- added R22: 1k, Resistor_SMD:R_0805_2012Metric, B.Cu at (174.0, 89.5)
- added R23: 1k, Resistor_SMD:R_0805_2012Metric, B.Cu at (174.0, 91.6)
- added R24: 200, Resistor_SMD:R_0402_1005Metric, F.Cu at (150.2, 78.6)
- added R25: 10, Resistor_SMD:R_0402_1005Metric, F.Cu at (154.3, 78.8)
- added R26: 1k, Resistor_SMD:R_0402_1005Metric, F.Cu at (149.7, 92.1)
- added R27: 10k, Resistor_SMD:R_0603_1608Metric, B.Cu at (122.2, 81.8)
- added SW2: SMD_4.2x3.2mm_h2.5mm, SparkFun-Switch:Push_SMD_4.2x3.2mm, B.Cu at (118.5, 86.2)
- added SW3: SMD_4.2x3.2mm_h2.5mm, SparkFun-Switch:Push_SMD_4.2x3.2mm, B.Cu at (118.5, 81.7)
- added U11: RP2350B, Package_DFN_QFN:QFN-80-1EP_10x10mm_P0.4mm_EP3.4x3.4mm, F.Cu at (149.4, 85.4)
- added U8: AP2112K-1.8, Package_TO_SOT_SMD:SOT-23-5, B.Cu at (178.1, 154.9)
- added U9: NE5532, Package_SO:SOIC-8_3.9x4.9mm_P1.27mm, B.Cu at (168.9, 94.3)
- added Y3: 32.768kHz, SparkFun-Clock:Crystal_SMD_3.2x1.5mm, F.Cu at (149.4, 94.1)
- C1, C2: value 22pF -> 47uF; footprint SparkFun-Capacitor:C_0402_1005Metric -> Capacitor_Tantalum_SMD:CP_EIA-7343-15_Kemet-W_HandSolder; moved to F.Cu
- C10, C7, C8, C9, D19, L1, Q2, R1, R11, R12, R13, R16, R3, R4, R5, R6, U3, U4: moved to B.Cu
- C16: value 1.0uF -> 0.1uF; footprint SparkFun-Capacitor:C_0603_1608Metric -> SparkFun-Capacitor:C_0402_1005Metric; moved to F.Cu
- C3, C4, U1, Y2: moved to F.Cu
- C5: value 47uF -> 1.0uF; footprint Capacitor_SMD:C_Elec_5x5.4 -> SparkFun-Capacitor:C_0805_2012Metric
- C6: value 47uF -> 2.2uF; footprint Capacitor_SMD:C_Elec_5x5.4 -> Capacitor_SMD:C_0402_1005Metric; moved to F.Cu
- R14, R15: value 1k -> 27; footprint SparkFun-Resistor:R_0603_1608Metric -> SparkFun-Resistor:R_0402_1005Metric; moved to F.Cu
- SW1: value MGB-SW1 -> SMD_4.2x3.2mm_h2.5mm
- U2: value RP2040 -> TLC5940PWP; footprint Package_DFN_QFN:QFN-56-1EP_7x7mm_P0.4mm_EP3.2x3.2mm -> Package_SO:HTSSOP-28-1EP_4.4x9.7mm_P0.65mm_EP2.85x5.4mm
- U6: value TEA5767 -> 74HC165; footprint TEA5767:TEA5767 -> SparkFun-Semiconductor-Standard:TSSOP-16_4.4x5mm_P0.65mm; moved to B.Cu
- moved ZOOM_CAP1 137.0 mm to (223.4, 68.1)
- moved D19 67.6 mm to (179.7, 147.5)
- moved R16 66.8 mm to (178.6, 145.1), turned to 0 degrees
- moved Q2 64.3 mm to (176.1, 143.2)
- moved R4 64.0 mm to (176.5, 147.5), turned to 90 degrees
- moved R13 64.0 mm to (178.1, 147.5), turned to -90 degrees
- moved C7 63.6 mm to (177.2, 150.8), turned to -90 degrees
- moved C9 61.3 mm to (179.2, 150.8), turned to 90 degrees
- moved R14 60.4 mm to (123.7, 72.7), turned to 0 degrees
- moved U4 59.7 mm to (174.5, 154.9), turned to -90 degrees
- moved R15 59.2 mm to (123.7, 73.7), turned to 0 degrees
- moved C10 58.8 mm to (174.5, 158.3), turned to 0 degrees
- moved U3 57.8 mm to (172.9, 147.5)
- moved C8 56.3 mm to (174.5, 151.4), turned to 180 degrees
- moved U6 55.9 mm to (159.4, 94.3), turned to -90 degrees
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Connections:
- C1 pad 1: GND -> +BATT
- C1 pad 2: Net-(U2-XIN) -> GND
- C16 pad 1: GND -> +3V3
- C16 pad 2: Net-(C16-Pad2) -> GND
- C2 pad 1: GND -> +BATT
- C2 pad 2: Net-(U2-XOUT) -> GND
- C5 pad 1: unconnected-(C5-Pad1) -> AFE_IN
- C5 pad 2: unconnected-(C5-Pad2) -> Net-(U9A-+)
- C6 pad 1: unconnected-(C6-Pad1) -> Net-(U11-ADC_AVDD)
- C6 pad 2: unconnected-(C6-Pad2) -> GND
- D1 pad 1: Net-(D1-K) -> GND
- D10 pad 1: Net-(D1-K) -> GND
- D11 pad 1: Net-(D1-K) -> GND
- D12 pad 1: Net-(D1-K) -> GND
- D13 pad 1: Net-(D1-K) -> GND
- D14 pad 1: Net-(D1-K) -> GND
- D15 pad 1: Net-(D1-K) -> GND
- D16 pad 1: Net-(D1-K) -> GND
- D17 pad 2: RGB_R -> Net-(D17-RA)
- D17 pad 3: RGB_G -> Net-(D17-GA)
- D17 pad 4: RGB_B -> Net-(D17-BA)
- D2 pad 1: Net-(D1-K) -> GND
- D2 pad 2: Net-(D10-A) -> Net-(D2-A)
- D3 pad 1: Net-(D1-K) -> GND
- D3 pad 2: Net-(D11-A) -> Net-(D3-A)
- D4 pad 1: Net-(D1-K) -> GND
- D4 pad 2: Net-(D12-A) -> Net-(D4-A)
- D5 pad 1: Net-(D1-K) -> GND
- D5 pad 2: Net-(D13-A) -> Net-(D5-A)
- D6 pad 1: Net-(D1-K) -> GND
- D6 pad 2: Net-(D14-A) -> Net-(D6-A)
- D7 pad 1: Net-(D1-K) -> GND
- D7 pad 2: Net-(D15-A) -> Net-(D7-A)
- D8 pad 1: Net-(D1-K) -> GND
- D8 pad 2: Net-(D16-A) -> Net-(D8-A)
- D9 pad 1: Net-(D1-K) -> GND
- D9 pad 2: Net-(D1-A) -> Net-(D9-A)
- R14 pad 1: GND -> USB_DP
- R15 pad 1: +3V3 -> USB_DM
- R15 pad 2: Net-(C16-Pad2) -> Net-(U11-USB_D-)
- SW1 pad P$1: N$15 -> (no net)
- SW1 pad P$3: N$11 -> (no net)
- SW1 pad P$C: SW -> (no net)
- SW1 pad P$MP1: GND -> (no net)
- SW1 pad P$MP2: GND -> (no net)
- U1 pad 14: unconnected-(U1-IOVDD1-Pad14) -> +3V3
- U1 pad 16: unconnected-(U1-DGND1-Pad16) -> GND
- U1 pad 19: unconnected-(U1-IOVDD2-Pad19) -> +3V3
- U1 pad 20: unconnected-(U1-DGND2-Pad20) -> GND
- U1 pad 21: unconnected-(U1-DGND3-Pad21) -> GND
- U1 pad 22: unconnected-(U1-DGND4-Pad22) -> GND
- U1 pad 24: unconnected-(U1-CVDD2-Pad24) -> +1V8
- U1 pad 31: unconnected-(U1-CVDD3-Pad31) -> +1V8
- U1 pad 32: unconnected-(U1-XTEST-Pad32) -> +3V3
- U1 pad 35: unconnected-(U1-GND-Pad35) -> GND
- U1 pad 37: unconnected-(U1-AGND0-Pad37) -> GNDA
- U1 pad 38: unconnected-(U1-AVDD0-Pad38) -> GNDA
- U1 pad 4: unconnected-(U1-DGND0-Pad4) -> GND
- U1 pad 40: unconnected-(U1-AGND1-Pad40) -> GNDA
- U1 pad 41: unconnected-(U1-AGND2-Pad41) -> GNDA
- U1 pad 43: unconnected-(U1-AVDD1-Pad43) -> VDDA
- U1 pad 45: unconnected-(U1-AVDD2-Pad45) -> VDDA
- U1 pad 47: unconnected-(U1-AGND3-Pad47) -> GNDA
- U1 pad 5: unconnected-(U1-CVDD0-Pad5) -> +1V8
- U1 pad 6: unconnected-(U1-IOVDD0-Pad6) -> +3V3
- U1 pad 7: unconnected-(U1-CVDD1-Pad7) -> +1V8
- U2 pad 1: Net-(U2-IOVDD-Pad1) -> GND
- U2 pad 10: Net-(U2-IOVDD-Pad1) -> Net-(D4-A)
- U2 pad 11: unconnected-(U2-GPIO8-Pad11) -> Net-(D5-A)
- U2 pad 12: unconnected-(U2-GPIO9-Pad12) -> Net-(D6-A)
- U2 pad 13: unconnected-(U2-GPIO10-Pad13) -> Net-(D7-A)
- U2 pad 14: unconnected-(U2-GPIO11-Pad14) -> Net-(D8-A)
- U2 pad 15: HSTX_12 -> Net-(D9-A)
- U2 pad 16: HSTX_13 -> Net-(D10-A)
- U2 pad 17: HSTX_14 -> Net-(D11-A)
- U2 pad 18: HSTX_15 -> Net-(D12-A)
- U2 pad 19: unconnected-(U2-TESTEN-Pad19) -> Net-(D13-A)
- U2 pad 20: Net-(U2-XIN) -> Net-(D14-A)
- U2 pad 21: Net-(U2-XOUT) -> Net-(D15-A)
- U2 pad 22: Net-(U2-IOVDD-Pad1) -> Net-(D16-A)
- U2 pad 23: Net-(U2-DVDD-Pad23) -> unconnected-(U2-XERR-Pad23)
- U2 pad 24: SWCLK -> unconnected-(U2-SOUT-Pad24)
- U2 pad 25: SWD -> unconnected-(U2-GSCLK-Pad25)
- U2 pad 27: HSTX_16 -> unconnected-(U2-IREF-Pad27)
- U2 pad 28: HSTX_17 -> +5V
- U2 pad 29: HSTX_18 -> GND
- U2 pad 4: SDA -> unconnected-(U2-SCLK-Pad4)
- U2 pad 5: SCL -> unconnected-(U2-SIN-Pad5)
- U2 pad 6: CODEC_SI -> unconnected-(U2-VPRG-Pad6)
- U2 pad 7: CODEC_CS -> Net-(D1-A)
- U2 pad 8: CODEC_SCLK -> Net-(D2-A)
- U2 pad 9: CODEC_SO -> Net-(D3-A)
- U6 pad 1: FM_SDA -> unconnected-(U6-~{PL}-Pad1)
- U6 pad 10: FM_ANT -> GND
- U6 pad 2: FM_SCL -> unconnected-(U6-CP-Pad2)
- U6 pad 3: GND -> BTN_L
- U6 pad 4: unconnected-(U6-W/R-Pad4) -> BTN_U
- U6 pad 5: +3V3 -> BTN_R
- U6 pad 6: GND -> BTN_D
- U6 pad 7: FM_R -> unconnected-(U6-~{Q7}-Pad7)
- U6 pad 8: FM_L -> GND
- U6 pad 9: unconnected-(U6-MPXO-Pad9) -> BTN_SR_OUT
Routing:
- net Net-(D9-A): track 0.00 -> 56.2 mm, vias 0 -> 1
- net Net-(D10-A): track 0.00 -> 50.2 mm, vias 0 -> 1
- net Net-(D1-A): track 0.00 -> 48.9 mm, vias 0 -> 1
- net Net-(D11-A): track 0.00 -> 44.9 mm, vias 0 -> 1
- net Net-(D2-A): track 0.00 -> 43.9 mm, vias 0 -> 1
- net Net-(D12-A): track 0.00 -> 38.8 mm, vias 0 -> 1
- net Net-(D3-A): track 0.00 -> 37.1 mm, vias 0 -> 1
- net Net-(D13-A): track 0.00 -> 32.9 mm, vias 0 -> 1
- net Net-(D4-A): track 0.00 -> 32.1 mm, vias 0 -> 1
- net Net-(D14-A): track 0.00 -> 26.6 mm, vias 0 -> 1
- net Net-(D5-A): track 0.00 -> 25.3 mm, vias 0 -> 1
- net +5V: track 0.00 -> 24.4 mm
- net FM_R: track 23.4 -> 0.00 mm
- net FM_L: track 20.7 -> 0.00 mm
- net Net-(D6-A): track 0.00 -> 17.4 mm, vias 0 -> 1
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Other:
- outline, holes or cut-outs redrawn
- board text removed: "CPU"
- board text removed: "RST BT0"
