File: stereoBoy/stereoBoy_MGB.kicad_sch (KiCad schematic)
At the start: 0 parts

Commit message: yeah
Changed lines of the file:
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@@
 	(paper "User" 455.651 299.872)
 	(sheet
-		(at 179.705 30.48)
-		(size 52.705 39.37)
+		(at 119.38 83.82)
+		(size 71.12 44.45)
 		(exclude_from_sim no)
 		(in_bom yes)
@@
 		)
 		(property "Sheetname" "stereoBoy_display"
-			(at 179.705 29.7684 0)
+			(at 119.38 83.1084 0)
 			(effects
 				(font
@@
 		)
 		(property "Sheetfile" "stereoBoy_display.kicad_sch"
-			(at 179.705 70.4346 0)
+			(at 119.38 128.8546 0)
 			(effects
 				(font
@@
 	)
 	(sheet
-		(at 38.735 23.8125)
-		(size 46.99 35.2425)
+		(at 41.91 31.75)
+		(size 71.12 44.45)
 		(exclude_from_sim no)
 		(in_bom yes)
@@
 		)
 		(property "Sheetname" "stereoBoy_power"
-			(at 38.735 23.1009 0)
+			(at 41.91 31.0384 0)
 			(effects
 				(font
@@
 		)
 		(property "Sheetfile" "stereoBoy_power.kicad_sch"
-			(at 38.735 59.6396 0)
+			(at 41.91 76.7846 0)
 			(effects
 				(font
@@
 		)
 		(property "Field2" ""
-			(at 38.735 23.8125 0)
+			(at 41.91 31.75 0)
 			(effects
 				(font
@@
 		)
 		(property "Field3" ""
-			(at 38.735 23.8125 0)
+			(at 41.91 31.75 0)
 			(effects
 				(font
@@
 	)
 	(sheet
-		(at 156.21 90.17)
-		(size 53.975 25.0825)
+		(at 41.91 135.89)
+		(size 71.12 44.45)
 		(exclude_from_sim no)
 		(in_bom yes)
@@
 		)
 		(property "Sheetname" "stereoBoy_input"
-			(at 156.21 89.4584 0)
+			(at 41.91 135.1784 0)
 			(effects
 				(font
@@
 		)
 		(property "Sheetfile" "stereoBoy_input.kicad_sch"
-			(at 156.21 115.8371 0)
+			(at 41.91 180.9246 0)
 			(effects
 				(font
@@
 	)
 	(sheet
-		(at 94.2975 25.7175)
-		(size 59.055 39.6875)
+		(at 119.38 31.75)
+		(size 71.12 44.45)
 		(exclude_from_sim no)
 		(in_bom yes)
@@
 		)
 		(property "Sheetname" "stereoBoy_audio"
-			(at 94.2975 25.0059 0)
+			(at 119.38 31.0384 0)
 			(effects
 				(font
@@
 		)
 		(property "Sheetfile" "stereoBoy_audio.kicad_sch"
-			(at 94.2975 65.9896 0)
+			(at 119.38 76.7846 0)
 			(effects
 				(font
@@
 	)
 	(sheet
-		(at 82.2325 82.55)
-		(size 53.975 25.0825)
+		(at 41.91 83.82)
+		(size 71.12 44.45)
 		(exclude_from_sim no)
 		(in_bom yes)
@@
 		)
 		(property "Sheetname" "stereoBoy_cpu"
-			(at 82.2325 81.8384 0)
+			(at 41.91 83.1084 0)
 			(effects
 				(font
@@
 		)
 		(property "Sheetfile" "stereoBoy_cpu.kicad_sch"
-			(at 82.2325 108.2171 0)
-			(effects
-				(font
+			(at 41.91 128.8546 0)
+			(effects
+				(font

Commit message: yuh
Changed lines of the file:
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@@
 	(paper "User" 455.651 299.872)
 	(sheet
-		(at 119.38 83.82)
+		(at 119.38 85.09)
 		(size 71.12 44.45)
 		(exclude_from_sim no)
@@
 		)
 		(property "Sheetname" "stereoBoy_display"
-			(at 119.38 83.1084 0)
-			(effects
-				(font
-					(size 1.27 1.27)
+			(at 119.38 84.3784 0)
+			(effects
+				(font
+					(size 3.81 3.81)
+					(thickness 0.762)
+					(bold yes)
 				)
 				(justify left bottom)
@@
 		)
 		(property "Sheetfile" "stereoBoy_display.kicad_sch"
-			(at 119.38 128.8546 0)
+			(at 119.38 130.1246 0)
 			(effects
 				(font
@@
 			(effects
 				(font
-					(size 1.27 1.27)
+					(size 3.81 3.81)
+					(thickness 0.762)
+					(bold yes)
 				)
 				(justify left bottom)
@@
 	)
 	(sheet
-		(at 41.91 135.89)
+		(at 41.91 138.43)
 		(size 71.12 44.45)
 		(exclude_from_sim no)
@@
 		)
 		(property "Sheetname" "stereoBoy_input"
-			(at 41.91 135.1784 0)
-			(effects
-				(font
-					(size 1.27 1.27)
+			(at 41.91 137.7184 0)
+			(effects
+				(font
+					(size 3.81 3.81)
+					(thickness 0.762)
+					(bold yes)
 				)
 				(justify left bottom)
@@
 		)
 		(property "Sheetfile" "stereoBoy_input.kicad_sch"
-			(at 41.91 180.9246 0)
+			(at 41.91 183.4646 0)
 			(effects
 				(font
@@
 			(effects
 				(font
-					(size 1.27 1.27)
+					(size 3.81 3.81)
+					(thickness 0.762)
+					(bold yes)
 				)
 				(justify left bottom)
@@
 	)
 	(sheet
-		(at 41.91 83.82)
+		(at 41.91 85.09)
 		(size 71.12 44.45)
 		(exclude_from_sim no)
@@
 		)
 		(property "Sheetname" "stereoBoy_cpu"
-			(at 41.91 83.1084 0)
-			(effects
-				(font
-					(size 1.27 1.27)
+			(at 41.91 84.3784 0)
+			(effects
+				(font
+					(size 3.81 3.81)
+					(thickness 0.762)
+					(bold yes)
 				)
 				(justify left bottom)
@@
 		)
 		(property "Sheetfile" "stereoBoy_cpu.kicad_sch"
-			(at 41.91 128.8546 0)
-			(effects
-				(font
+			(at 41.91 130.1246 0)
+			(effects
+				(font
