File: stereoBoy/stereoBoy_audio.kicad_sch (KiCad schematic)
At the start: 15 parts, among them J5 SJ1-3524N, U1 CODECODER-VS1053B_LQFP48_, U16 PAM8302AAD, U5 TS5A23159DGS, U6 TEA5767, U7 TS5A23159DGS, Y2 12M

Commit message: yeah
Parts:
- removed C5, C6: 47uF, Capacitor_SMD:C_Elec_5x5.4, symbol SparkFun-Capacitor:47uF_6.6x6.6_50V_20%
- removed U6: TEA5767, TEA5767:TEA5767, symbol TEA5767:TEA5767
- added C5: 1.0uF, SparkFun-Capacitor:C_0805_2012Metric, symbol SparkFun-Capacitor:1.0uF_0805_25V_10%
- added R20, R21, R22, R23: 1k, Resistor_SMD:R_0805_2012Metric, symbol SparkFun-Resistor:R
- added U9: NE5532, Package_SO:SOIC-8_3.9x4.9mm_P1.27mm, symbol Amplifier_Operational:NE5532
Connections:
- net +3V3: now also U1.14 (IOVDD1), U1.19 (IOVDD2), U1.32 (XTEST), U1.6 (IOVDD0), R20.1
- net GND: now also U1.16 (DGND1), U1.20 (DGND2), U1.21 (DGND3), U1.22 (DGND4), U1.35 (GND), U1.4 (DGND0), R21.2, R23.2
- net +1V8: now reaches U1.24 (CVDD2)
- net +1V8: now also U1.31 (CVDD3), U1.5 (CVDD0), U1.7 (CVDD1)
- net GNDA: now reaches U1.37 (AGND0)
- net GNDA: now also U1.38 (AVDD0), U1.40 (AGND1), U1.41 (AGND2), U1.47 (AGND3)
- net VDDA: now reaches U1.43 (AVDD1)
- net VDDA: now also U1.45 (AVDD2)
- new net: C5.2, R20.2, R21.1, U9.3 (+)
- new net: R22.2, R23.1, U9.2 (-)
- new net AFE_IN: C5.1
- new net AFE_OUT: R22.1, U9.1

Commit message: yuh
Parts:
- removed C31: 1.0uF, SparkFun-Capacitor:C_0603_1608Metric, symbol SparkFun-Capacitor:1.0uF_0603_16V_10%
- removed C5: 1.0uF, SparkFun-Capacitor:C_0805_2012Metric, symbol SparkFun-Capacitor:1.0uF_0805_25V_10%
- removed J5: SJ1-3524N, SJ1-3524N:SJ1-3524N, symbol SJ1-3524N:SJ1-3524N
- removed R30, R31: 1k, SparkFun-Resistor:R_0603_1608Metric, symbol SparkFun-Resistor:1k_0603
- removed U16: PAM8302AAD, Package_SO:MSOP-8_3x3mm_P0.65mm, symbol Amplifier_Audio:PAM8302AAD
- removed U5, U7: TS5A23159DGS, Package_SO:VSSOP-10_3x3mm_P0.5mm, symbol Analog_Switch:TS5A23159DGS
- removed U9: NE5532, Package_SO:SOIC-8_3.9x4.9mm_P1.27mm, symbol Amplifier_Operational:NE5532
- added C13: 1.0uF, Capacitor_SMD:C_0603_1608Metric, symbol SparkFun-Capacitor:1.0uF_0805_25V_10%
- added C24, C31, C41: 1.0uF, Capacitor_SMD:C_0402_1005Metric, symbol SparkFun-Capacitor:1.0uF_0805_25V_10%
- added C26, C27, C37, C38, C39, C40, C71: 1.0uF, SparkFun-Capacitor:C_0402_1005Metric, symbol SparkFun-Capacitor:0.1uF_0402_16V_10%
- added C32, C33: 100uF, SparkFun-Capacitor:C_1206_3216Metric, symbol SparkFun-Capacitor:100uF_1206_50V_10%
- added C34, C53, C61, C64, C69, C70: 1.0uF, Capacitor_SMD:C_0805_2012Metric, symbol SparkFun-Capacitor:1.0uF_0805_25V_10%
- added C35: 0.1uF, SparkFun-Capacitor:C_0805_2012Metric, symbol SparkFun-Capacitor:1.0uF_0805_25V_10%
- added C36, C52, C66, C67, C72, C73, C74: 1.0uF, Capacitor_SMD:C_1206_3216Metric, symbol SparkFun-Capacitor:1.0uF_0805_25V_10%
- added C45, C46, C5, C55: 0.1uF, SparkFun-Capacitor:C_0402_1005Metric, symbol SparkFun-Capacitor:10uF_0603_10V_20%
- added C49: 1uF, SparkFun-Capacitor:C_0603_1608Metric, symbol SparkFun-Capacitor:1.0uF_0805_25V_10%
- added C50: 47nF, SparkFun-Capacitor:C_0402_1005Metric, symbol SparkFun-Capacitor:1.0uF_0805_25V_10%
- added C51: 1.0uF, SparkFun-Capacitor:C_0402_1005Metric, symbol SparkFun-Capacitor:1.0uF_0805_25V_10%
- added C54: 0.1uF, SparkFun-Capacitor:C_0603_1608Metric, symbol SparkFun-Capacitor:1.0uF_0805_25V_10%
- added C56: 4.7uF, SparkFun-Capacitor:C_0805_2012Metric, symbol SparkFun-Capacitor:1.0uF_0805_25V_10%
- added C62, C65: 1.0uF, SparkFun-Capacitor:C_0603_1608Metric, symbol SparkFun-Capacitor:1.0uF_0805_25V_10%
- added C75: 0.1uF, SparkFun-Capacitor:C_0402_1005Metric, symbol SparkFun-Capacitor:1.0uF_0805_25V_10%
- added J5: SJ-43514, SJ_43514:SJ_43514, symbol SJ-43514:SJ-43514
- added L8: 600Ω @ 100MHz, Capacitor_SMD:C_0603_1608Metric, symbol SparkFun-Coil:Ferrite_600Ohm_0805_500mA
- added R30: 10K, Resistor_SMD:R_0402_1005Metric, symbol SparkFun-Resistor:470_0402
- added R34, R39, R57: 10k, Resistor_SMD:R_0402_1005Metric, symbol SparkFun-Resistor:R
- added R40: 7.2K, Resistor_SMD:R_0402_1005Metric, symbol SparkFun-Resistor:R
- added R50: 100K, Resistor_SMD:R_0402_1005Metric, symbol SparkFun-Resistor:470_0402
- added R51: 1M, Resistor_SMD:R_0402_1005Metric, symbol SparkFun-Resistor:470_0402
- added R52: 10, Resistor_SMD:R_0402_1005Metric, symbol SparkFun-Resistor:470_0402
- added R53: 2.2k, Resistor_SMD:R_0603_1608Metric, symbol SparkFun-Resistor:470_0402
- added TP10, TP27, TP31, TP32, TP33: TestPoint_Alt, TestPoint:TestPoint_Pad_D1.0mm, symbol Connector:TestPoint_Alt
- added U10: TLV320AIC3100, Package_DFN_QFN:VQFN-32-1EP_5x5mm_P0.5mm_EP3.5x3.5mm, symbol Audio:TLV320AIC3100
- added U13: REF2033, Package_TO_SOT_SMD:SOT-23-5, symbol Reference_Voltage:REF2033
- added U9: OPA1678, Package_SO:SOIC-8_3.9x4.9mm_P1.27mm, symbol Amplifier_Operational:OPA1678
- C3, C4: value 22pF -> 33pF
- R20: value 1k -> 10k; footprint Resistor_SMD:R_0805_2012Metric -> Resistor_SMD:R_0402_1005Metric; now not fitted
- R21: value 1k -> 7.2K; footprint Resistor_SMD:R_0805_2012Metric -> Resistor_SMD:R_0402_1005Metric; now not fitted
- R22, R23: value 1k -> 10K; footprint Resistor_SMD:R_0805_2012Metric -> Resistor_SMD:R_0402_1005Metric; now not fitted
- Y2: value 12M -> 12.288M
Connections:
- net +1V8: now also C24.2, C26.2, C31.2, C39.2, C40.2, U10.3 (DVDD)
- net +3V3: now also C13.2, C27.2, C34.2, C35.1, C37.2, C38.2, C41.2, C51.1, C52.2, C53.2, C56.1, C61.2, C66.2, C67.2, C69.2, C70.2, C71.2, C72.2, C73.2, C74.2, L8.1, R30.2, U10.17 (AVDD), U10.2 (IOVDD), U10.28 (HPVDD), U13.3 (EN), U13.4 (IN), U9.8 (V+); no longer R20.1
- net AFE_OUT: now also C45.2, C55.2; no longer R22.1
- net CODEC_L_OUT: now also R20.2
- net CODEC_R_OUT: now also R39.2
- net GND: now also U1.37 (AGND0), U1.40 (AGND1), U1.41 (AGND2), U1.47 (AGND3), C13.1, C24.1, C26.1, C27.1, C31.1, C34.1, C35.2, C36.1, C37.1, C38.1, C39.1, C40.1, C41.1, C50.1, C51.2, C52.1, C53.1, C54.2, C56.2, C61.1, C62.1, C64.1, C65.2, C66.1, C67.1, C69.1, C70.1, C71.1, C72.1, C73.1, C74.1, C75.2, J5.4, R50.2, U10.1 (IOVSS), U10.13 (MIC1LP), U10.14 (MIC1RP), U10.16 (AVSS), U10.18 (DVSS), U10.20 (SPKVSS), U10.25 (SPKVSS), U10.29 (HPVSS), U10.33 (EP), U13.2 (GND), U9.4 (V-); no longer R21.2, R23.2
- net I2S_BCLK: now reaches U1.11 (GPIO6/I2S_SCLK3)
- net I2S_BCLK: now also U10.7 (BCLK)
- net I2S_DIN: now reaches U1.12 (GPIO7/I2S_SDATA3)
- net I2S_DIN: now also U10.5 (DIN)
- net CODEC_XDCS: now reaches U1.13 (XDCS/BSYNC1)
- net CODEC_XDCS: now also TP32.1
- net at C3.2, U1.17 (XTALO), Y2.1: now also R51.2
- net at C4.2, U1.18 (XTALI), Y2.2: now also R51.1
- net CODEC_XCS: now reaches U1.23 (XCS)
- net CODEC_XCS: now also TP33.1
- net I2S_MCLK: now reaches U1.25 (GPIO/I2S_MCLK3)
- net I2S_MCLK: now also U10.8 (MCLK)
- net CODEC_RX: now reaches U1.26 (RX)
- net CODEC_TX: now reaches U1.27 (TX)
- net CODEC_RST: now reaches U1.3 (XRESET)
- net CODEC_RST: now also R50.1, TP27.1
- net I2S_WSEL: now reaches U1.36 (GPIO4/I2S-LROUT3)
- net I2S_WSEL: now also U10.6 (WCLK)
- net GBUF: now reaches U1.42 (GBUF)
- net GBUF: now also C49.2, R52.2
- net at U1.44 (RCAP): now also C49.1
- net CODEC_DREQ: now reaches U1.8 (DREQ)
- net CODEC_DREQ: now also TP31.1
- net at R21.1: now also R57.2, U9.1; no longer R20.2
- net at R23.1: now also U9.5 (+); no longer R22.2
- net CODEC_SCLK renamed SPI1_SCK
- net CODEC_SI renamed SPI1_MOSI
- net CODEC_SO renamed SPI1_MISO
- removed net GNDA: U1.37 (AGND0), U1.38 (AVDD0), U1.40 (AGND1), U1.41 (AGND2), U1.47 (AGND3)
- net SPK+: no longer names the net of SPK_CONN1.1 (Pin_1)
- net SPK+: now also U10.22 (SPKP), U10.26 (SPKP)
- net SPK-: no longer names the net of SPK_CONN1.2 (Pin_2)
- net SPK-: now also U10.19 (SPKM), U10.23 (SPKM)
- net VDDA renamed AVDD
- net AVDD: now also U1.38 (AVDD0), C54.1, C75.1, L8.2, TP10.1
- new net: C5.1, R20.1
- new net: C5.2, R21.2, U9.2 (-)
- new net: C33.2, U10.30 (HPR)
- new net: C45.1, R34.1
- new net: R34.2, R40.1, U9.7
- new net: C50.2, R52.1
- new net: C55.1, R57.1
- new net: C46.2, R40.2, U9.6 (-)
- new net: R22.1, U9.3 (+)
- new net: C46.1, R39.1
- new net: C32.1, U10.27 (HPL)
- new net +5V: C64.2
- new net +5V_SPK: C36.2, C62.2, C65.1, U10.21 (SPKVDD), U10.24 (SPKVDD)
- new net ADC_VREF: U13.5 (Vref)
- new net AFE_VBIAS: R22.2, R23.2, U13.1 (Vbias)
- new net DAC_GPIO1: U10.32 (GPIO1)
- new net DAC_RST: R30.1, U10.31 (~{RESET})
- new net HP_L: C32.2, J5.2
- new net HP_R: C33.1, J5.3
- new net I2C0_SCL: U10.10 (SCL)
- new net I2C0_SDA: U10.9 (SDA)
- new net MICBIAS: R53.2, U10.12 (MICBIAS)
- new net MICDET: J5.1, R53.1, U10.11 (VOL/MICDET)
- no-connect marks 0 -> 4
Other:
- note added: "AFE options: -> jumper to select left, right, or mono"
- note added: "Analog Front-End (AFE)"
- note added: "Audio Co-processor"
- note added: "Based on Adafruit TLV320DAC3100 schematic"
- note added: "Based on Adafruit VS1053B schematic"
- note added: "Converts stereo audio into DC-biased mono signal"
- note added: "DAC"
- note added: "Decoupling capacitors"
- note added: "Final audio output stage"
- note added: "Jumpers for SPKVDD select"
- note added: "NOT NEEDED (I think)"
- note added: "POWER DECOUPLING"
- note added: "STEREOBOY"
- note added: "STEREOBOY AUDIO"
- note added: "Tested with Adafruit TLV320DAC3100 breakout connected to VS1053B with I2S and RP2350 with I2C (SCL=21 SDA=20)"
- note added: "Tested with Adafruit VS1053B breakout board using SD card and codec on same SPI bus"
- note added: "VS1053 analog output is biased at 1.25V"
- note added: "VS1053B CODEC"
- note added: "Verified!"
- note added: "Verified! (Headphones, speaker, headphone det.)"
- note added: "with simulation + breadboard prototype & TL082 & resistor divide 1.65 Vbias"
- moved on the sheet: C3, C4, SPK_CONN1, U1, Y2

Commit message: yuh
Other:
- moved on the sheet: C13, C24, C26, C27, C3, C31, C34, C35, C36, C37, C38, C39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
