File: stereoBoy/stereoBoy_display.kicad_sch (KiCad schematic)
At the start: 21 parts, among them Q1 DMG2301L

Commit message: yeah
Parts:
- added J1: Conn_01x22_FPC_0.5mm, SparkFun-Connector:FPC_1x22_P0.5mm_Horizontal_BottomContact, symbol SparkFun-Connector:Conn_01x22_FPC_P0.5mm_Horizontal_BottomContact
- added R17, R18, R19: 330, SparkFun-Resistor:R_0603_1608Metric, symbol SparkFun-Resistor:330_0603
- added U2: TLC5940PWP, Package_SO:HTSSOP-28-1EP_4.4x9.7mm_P0.65mm_EP2.85x5.4mm, symbol Driver_LED:TLC5940PWP
Connections:
- net GND: now also D1.1 (K), D10.1 (K), D11.1 (K), D12.1 (K), D13.1 (K), D14.1 (K), D15.1 (K), D16.1 (K), D2.1 (K), D3.1 (K), D4.1 (K), D5.1 (K), D6.1 (K), D7.1 (K), D8.1 (K), D9.1 (K), U2.1 (GND), U2.29 (PAD)
- net RGB_B: now also R19.2; no longer D17.4 (BA)
- net RGB_G: now also R18.2; no longer D17.3 (GA)
- net RGB_R: now also R17.2; no longer D17.2 (RA)
- net at D10.2 (A): now also U2.16 (OUT9); no longer D2.2 (A)
- net at D14.2 (A): now also U2.20 (OUT13); no longer D6.2 (A)
- net at D4.2 (A): now also U2.10 (OUT3); no longer D12.2 (A)
- net at D5.2 (A): now also U2.11 (OUT4); no longer D13.2 (A)
- net at D7.2 (A): now also U2.13 (OUT6); no longer D15.2 (A)
- net at D8.2 (A): now also U2.14 (OUT7); no longer D16.2 (A)
- net at D11.2 (A): now also U2.17 (OUT10); no longer D3.2 (A)
- net at D9.2 (A): now also U2.15 (OUT8); no longer D1.2 (A)
- new net: D17.2 (RA), R17.1
- new net: D17.3 (GA), R18.1
- new net: D17.4 (BA), R19.1
- new net: D13.2 (A), U2.19 (OUT12)
- new net: D3.2 (A), U2.9 (OUT2)
- new net: D15.2 (A), U2.21 (OUT14)
- new net: D16.2 (A), U2.22 (OUT15)
- new net: D12.2 (A), U2.18 (OUT11)
- new net: D6.2 (A), U2.12 (OUT5)
- new net: D1.2 (A), U2.7 (OUT0)
- new net: D2.2 (A), U2.8 (OUT1)
- new net +5V: U2.28 (VCC)
Other:
- moved on the sheet: D1, D10, D11, D12, D13, D14, D15, D16, D2, D3, D4, D5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

Commit message: yuh
Parts:
- removed J1: Conn_01x22_FPC_0.5mm, SparkFun-Connector:FPC_1x22_P0.5mm_Horizontal_BottomContact, symbol SparkFun-Connector:Conn_01x22_FPC_P0.5mm_Horizontal_BottomContact
- removed LS1: CBT-09427-SMT, CBT_09427_SMT_TR:CBT_09427_SMT_TR, symbol CBT_09427_SMT_TR:CBT-09427-SMT
- removed U2: TLC5940PWP, Package_SO:HTSSOP-28-1EP_4.4x9.7mm_P0.65mm_EP2.85x5.4mm, symbol Driver_LED:TLC5940PWP
- added BZ1: Buzzer, Buzzer_Beeper:Buzzer_CUI_CPT-9019S-SMT, symbol Device:Buzzer
- added C29: 1.0uF, SparkFun-Capacitor:C_0805_2012Metric, symbol SparkFun-Capacitor:1.0uF_0805_25V_10%
- added C43: 10uF, Capacitor_SMD:CP_Elec_6.3x4.5, symbol SparkFun-Capacitor:10uF_0603_6.3V_20%_Polar(Tant)
- added J1: Conn_01x12, 1.54_IPS_LCD_Adafruit:1.54_IPS_FPC_Solder, symbol SparkFun-Connector:Conn_01x12_P2.54mm
- added J6: Conn_01x09, SparkFun-Connector:1x09_P2.54mm, symbol SparkFun-Connector:Conn_01x09_P2.54mm
- added Q3: BSS138, Package_TO_SOT_SMD:SOT-23, symbol Transistor_FET:BSS138
- added R28: 10, SparkFun-Resistor:R_0603_1608Metric, symbol SparkFun-Resistor:1k_0603
- added R29: 10k, SparkFun-Resistor:R_0603_1608Metric, symbol SparkFun-Resistor:1k_0603
- added R31: 1k, SparkFun-Resistor:R_0603_1608Metric, symbol SparkFun-Resistor:1k_0603
- added TP1, TP2: TestPoint_Alt, TestPoint:TestPoint_Pad_D1.0mm, symbol Connector:TestPoint_Alt
- added U2: PCA9685PW, Package_SO:TSSOP-28_4.4x9.7mm_P0.65mm, symbol Driver_LED:PCA9685PW
- added U5: APX803, Package_TO_SOT_SMD:SOT-23, symbol Power_Supervisor:LM810
Connections:
- net +5V: now also C29.2, C43.1, U2.28 (VDD)
- net GND: now also BZ1.2 (-), C29.1, C43.2, J1.1 (Pin_1), J1.12 (Pin_12), J1.5 (Pin_5), J1.6 (Pin_6), J6.8 (Pin_8), J6.9 (Pin_9), Q3.2 (S), U2.1 (A0), U2.14 (VSS), U2.2 (A1), U2.23 (~{OE}), U2.24 (A5), U2.3 (A2), U2.4 (A3), U2.5 (A4), U5.1 (GND)
- net at D10.2 (A): now also U2.16 (LED9)
- net at D14.2 (A): now also U2.20 (LED13)
- net at D4.2 (A): now also U2.9 (LED3)
- net at D5.2 (A): now also U2.10 (LED4)
- net at D13.2 (A): now also U2.19 (LED12)
- net at D7.2 (A): now also U2.12 (LED6)
- net at D8.2 (A): now also U2.13 (LED7)
- net at D11.2 (A): now also U2.17 (LED10)
- net at D18.1 (K), Q1.2 (S): now also BZ1.1 (+)
- net at D3.2 (A): now also U2.8 (LED2)
- net at D15.2 (A): now also U2.21 (LED14)
- net at D16.2 (A): now also U2.22 (LED15)
- net at D9.2 (A): now also U2.15 (LED8)
- net at D12.2 (A): now also U2.18 (LED11)
- net at D6.2 (A): now also U2.11 (LED5)
- net at D1.2 (A): now also U2.6 (LED0)
- net at D2.2 (A): now also U2.7 (LED1)
- net +3.3V renamed +3V3
- net +3V3: now also J1.3 (Pin_3), J1.4 (Pin_4), J6.6 (Pin_6), R29.2, U5.3 (VCC)
- new net: Q3.1 (G), R29.1, R31.1
- new net: Q3.3 (D), R28.1
- new net BACKLIGHT: J6.7 (Pin_7), R31.2
- new net I2C1_SCL: TP1.1, U2.26 (SCL)
- new net I2C1_SDA: TP2.1, U2.27 (SDA)
- new net LEDK: J1.2 (Pin_2), R28.2
- new net SPI0_CS: J1.8 (Pin_8), J6.4 (Pin_4)
- new net SPI0_MISO: J6.1 (Pin_1)
- new net SPI0_MOSI: J1.10 (Pin_10), J6.2 (Pin_2)
- new net SPI0_SCK: J1.9 (Pin_9), J6.3 (Pin_3)
- new net TFTDC_3V: J1.7 (Pin_7)
- new net TFTRST_3V: J1.11 (Pin_11), J6.5 (Pin_5), U5.2 (RESET)
Other:
- note added: "1.54" IPS LCD"
- note added: "PCA9685 LED DRIVER"
- note added: "PIEZO BUZZER"
- note added: "RGB LED"
- note added: "STEREOBOY"
- note added: "STEREOBOY DISPLAY"
- note added: "Verified!"
- note added: "with PCA9685 IC on breadboard"
- moved on the sheet: D1, D10, D11, D12, D13, D14, D15, D16, D17, D18, D2, D3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

Commit message: yuh
Parts:
- removed D17: RGB, LED_SMD:LED_WS2812B-Mini_PLCC4_3.5x3.5mm, symbol Device:LED_KRGB
- added D17: CLMVC-FKA-CL1D1L71BB7C3C3, CREE_LED_2mm_x_2mm_Common_Anode:CREE_LED_2mm_x_2mm_Common_Anode, symbol CREE_LED_2mm_x_2mm_Common_Anode:CLMVC-FKA-CL1D1L71BB7C3C3
- added R32, R58, R59, R60, R61, R62, R63, R64, R65, R66, R67, R68, R69, R70, R71, R72: 220, SparkFun-Resistor:R_0402_1005Metric, symbol SparkFun-Resistor:220_0402
- R17, R18, R19: footprint SparkFun-Resistor:R_0603_1608Metric -> SparkFun-Resistor:R_0402_1005Metric
Connections:
- net +3V3: now also D17.1
- net at D10.2 (A): now also R66.2; no longer U2.16 (LED9)
- net at R17.1: now also D17.2
- net at R18.1: now also D17.3
- net at R19.1: now also D17.4
- net at D14.2 (A): now also R70.2; no longer U2.20 (LED13)
- net at U2.9 (LED3): now also R60.1; no longer D4.2 (A)
- net at D5.2 (A): now also R61.2; no longer U2.10 (LED4)
- net at U2.19 (LED12): now also R69.1; no longer D13.2 (A)
- net at D7.2 (A): now also R63.2; no longer U2.12 (LED6)
- net at D8.2 (A): now also R64.2; no longer U2.13 (LED7)
- net at U2.11 (LED5): now also R62.1; no longer D6.2 (A)
- net at U2.15 (LED8): now also R65.1; no longer D9.2 (A)
- net at U2.17 (LED10): now also R67.1; no longer D11.2 (A)
- net at U2.18 (LED11): now also R68.1; no longer D12.2 (A)
- net at U2.21 (LED14): now also R71.1; no longer D15.2 (A)
- net at U2.22 (LED15): now also R72.1; no longer D16.2 (A)
- net at U2.6 (LED0): now also R32.1; no longer D1.2 (A)
- net at U2.7 (LED1): now also R58.1; no longer D2.2 (A)
- net at U2.8 (LED2): now also R59.1; no longer D3.2 (A)
- new net: D4.2 (A), R60.2
- new net: D13.2 (A), R69.2
- new net: D1.2 (A), R32.2
- new net: R70.1, U2.20 (LED13)
- new net: D12.2 (A), R68.2
- new net: D16.2 (A), R72.2
- new net: R61.1, U2.10 (LED4)
- new net: R63.1, U2.12 (LED6)
- new net: R64.1, U2.13 (LED7)
- new net: R66.1, U2.16 (LED9)
- new net: D11.2 (A), R67.2
- new net: D3.2 (A), R59.2
- new net: D15.2 (A), R71.2
- new net: D9.2 (A), R65.2
- new net: D6.2 (A), R62.2
- new net: D2.2 (A), R58.2
Other:
- moved on the sheet: R17, R18, R19
