File: GameBoy_Pocket_Original_Files/MGBC-MBL-01_2_1.kicad_pcb (KiCad board)
At the start: 2 copper layers, 69.6 x 114.8 mm, 130 parts, among them P1 MGB-CART, P2 GBC_LCDH, P3 LINKPORTDMG-LINK-SHORT, P4 MGB-PWRJACK, P5 MGBHPMGB, Q1 BSS84, SW0 TPTP20R, SW1 MGB-SW1, SW2 NAV_SWITCH, U1 GBC_CPU, U2 LH52256CVTXIZ, U3 LM4853, U4 TLV70233QDBVRQ1, U5 MGB-PWR_BD, U6 TPS3840, U7 TL331, X1 8.388608MHZ12SMX-B-4-PAD

Commit message: yuh
Parts:
- added C48: 1uF, MGBC-MBL-01_2_1:C0603, F.Cu at (220.3, 52.7)
Routing:
- net (no net): track 0.00 -> 48.1 mm, vias 0 -> 366
- net N$15: track 22.8 -> 1.03 mm, vias 9 -> 0
- net GND: track 175.6 -> 162.9 mm, vias 311 -> 28
- net EM10_GND: track 16.2 -> 3.81 mm
- net BATT: track 0.76 -> 0.00 mm, vias 25 -> 0
- net SW1B: track 35.7 -> 35.2 mm, vias 8 -> 0
- net SW: vias 13 -> 8
- net EM10_POS: vias 5 -> 0
- net +5V: vias 32 -> 1
- added copper zone on B.Cu, net (none)
- added copper zone on F.Cu, net (none)
- removed copper zone on F.Cu, net +3V3
- removed copper zone on B.Cu, net +5V
- removed copper zone on F.Cu, net +5V
- removed copper zone on B.Cu, net BATT
- removed copper zone on F.Cu, net BATT
- removed copper zone on F.Cu, net EM10_GND
- removed copper zone on B.Cu, net EM10_POS
- removed copper zone on F.Cu, net EM10_POS
- removed copper zone on B.Cu, net GND
- removed copper zone on F.Cu, net GND
- removed copper zone on F.Cu, net N$12
- removed copper zone on F.Cu, net N$13
- removed copper zone on B.Cu, net N$15
- removed copper zone on F.Cu, net N$15
- removed copper zone on F.Cu, net N$16
- removed copper zone on F.Cu, net N$17
- removed copper zone on F.Cu, net N$20
- removed copper zone on B.Cu, net SW
- removed copper zone on F.Cu, net SW
- removed copper zone on B.Cu, net SW1B
- removed copper zone on F.Cu, net SW1B
