File: stereoMag/stereoMag_devKit/stereoMag.kicad_pcb (KiCad board)
At the start: 2 copper layers, 51 x 60.7 mm, 21 parts, among them J1 GameBoy_GamePak_CGB-002, J2 TSM-110-01-S-DH-LC, J6 microSD, SW1 SPDT_Slide_SMD_6.7x2.6mm, U1 W25Q16JVSS, U2 FM24C64B, U3 W25Q16JVSS

Commit message: New thingies
Parts:
- removed SW1: SPDT_Slide_SMD_6.7x2.6mm, SparkFun-Switch:Slide_SPST_SMD_6.7x2.6mm
- removed U3: W25Q16JVSS, Package_SO:SOIC-8_5.3x5.3mm_P1.27mm
- added U4: PSRAM, Package_SO:SOIC-8_3.9x4.9mm_P1.27mm, F.Cu at (134.1, 110.3)
- C1, C2: footprint Capacitor_SMD:CP_Elec_5x3 -> Capacitor_SMD:C_1206_3216Metric
- U1: value W25Q16JVSS -> FLASH; footprint Package_SO:SOIC-8_5.3x5.3mm_P1.27mm -> Package_SO:SOIC-8_3.9x4.9mm_P1.27mm
- moved U2 2.25 mm to (161.1, 113.3)
- moved C1 1.91 mm to (168.8, 112.2)
- moved C7 1.27 mm to (129.5, 111.3)
- moved C8 1.27 mm to (129.5, 117.5)
Connections:
- J1 pad 10: ADC1 -> SD_DETECT
- J1 pad 7: QSPI_CS -> QSPI_CS0
- J1 pad 8: SD_DETECT -> SD_CS
- J1 pad 9: SD_CS -> QSPI_CS1
- U1 pad 1: F0_CS -> QSPI_CS0
- U2 pad 1: unconnected-(U2-A0-Pad1) -> +3V3
- U2 pad 2: unconnected-(U2-A1-Pad2) -> GND
- U2 pad 3: unconnected-(U2-A2-Pad3) -> GND
- U2 pad 4: unconnected-(U2-VSS-Pad4) -> GND
- U2 pad 5: unconnected-(U2-SDA-Pad5) -> I2C0_SDA
- U2 pad 6: unconnected-(U2-SCL-Pad6) -> I2C0_SCL
- U2 pad 7: unconnected-(U2-WP-Pad7) -> GND
- U2 pad 8: unconnected-(U2-VDD-Pad8) -> +3V3
Routing:
- net ADC1: track 38.1 -> 0.00 mm, vias 1 -> 0
- net QSPI_CS: track 31.1 -> 0.00 mm
- net F0_CS: track 23.8 -> 0.00 mm
- net F1_CS: track 21.1 -> 0.00 mm, vias 2 -> 0
- net QSPI_CS1: track 0.00 -> 12.5 mm
- net +3V3: track 127.8 -> 138.3 mm
- net GND: track 6.01 -> 14.8 mm, vias 6 -> 8
- net I2C0_SCL: track 47.4 -> 55.2 mm, vias 0 -> 1
- net I2C0_SDA: track 46.1 -> 53.8 mm, vias 0 -> 1
- net QSPI_CS0: track 0.00 -> 5.23 mm
- net QSPI_SCK: track 19.3 -> 16.4 mm
- net QSPI_D1: track 16.2 -> 14.1 mm
- net QSPI_D2: track 18.1 -> 16.0 mm
- net SD_CS: track 40.7 -> 38.8 mm, vias 0 -> 1
- net SD_DETECT: track 37.4 -> 36.2 mm
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Other:
- board text removed: "0"
- board text removed: "1"
- board text removed: "DUOFLASH"
- board text removed: "™"
